File: SBR001-202.kicad_pcb (KiCad board)
At the start: 2 copper layers, 895.4 x 10.9 mm, 80 parts

Commit message: Schematic and layout complete and ready for review
Parts:
- added D1001: GRN, LEDs:LED_0603, F.Cu at (843.6, 58.4)
- added D1002: GRN, LEDs:LED_0603, F.Cu at (869.0, 58.5)
- added D1003: GRN, LEDs:LED_0603, F.Cu at (889.0, 58.4)
- added D1004: GRN, LEDs:LED_0603, F.Cu at (848.2, 58.4)
- added D1005: GRN, LEDs:LED_0603, F.Cu at (853.3, 58.4)
- added D1006: GRN, LEDs:LED_0603, F.Cu at (858.5, 58.4)
- added D1007: GRN, LEDs:LED_0603, F.Cu at (863.6, 58.5)
- added D1008: GRN, LEDs:LED_0603, F.Cu at (874.0, 58.5)
- added D1009: GRN, LEDs:LED_0603, F.Cu at (878.8, 58.5)
- added D1010: GRN, LEDs:LED_0603, F.Cu at (883.8, 58.4)
- added D1011: GRN, LEDs:LED_0603, F.Cu at (894.3, 58.4)
- added D1012: GRN, LEDs:LED_0603, F.Cu at (899.2, 58.5)
- added D1013: GRN, LEDs:LED_0603, F.Cu at (909.0, 58.5)
- added D1015: GRN, LEDs:LED_0603, F.Cu at (903.9, 58.5)
- added D1016: GRN, LEDs:LED_0603, F.Cu at (913.0, 58.5)
- added D1017: GRN, LEDs:LED_0603, F.Cu at (917.8, 58.5)
- added D1101: GRN, LEDs:LED_0603, B.Cu at (31.6, 58.5)
- added D1102: GRN, LEDs:LED_0603, B.Cu at (56.8, 58.5)
- added D1103: GRN, LEDs:LED_0603, B.Cu at (76.7, 58.5)
- added D1104: GRN, LEDs:LED_0603, B.Cu at (36.2, 58.5)
- added D1105: GRN, LEDs:LED_0603, B.Cu at (41.0, 58.5)
- added D1106: GRN, LEDs:LED_0603, B.Cu at (46.0, 58.5)
- added D1107: GRN, LEDs:LED_0603, B.Cu at (51.3, 58.7)
- added D1108: GRN, LEDs:LED_0603, B.Cu at (61.7, 58.5)
- added D1109: GRN, LEDs:LED_0603, B.Cu at (66.7, 58.5)
- added D1110: GRN, LEDs:LED_0603, B.Cu at (71.5, 58.5)
- added D1111: GRN, LEDs:LED_0603, B.Cu at (82.0, 58.5)
- added D1112: GRN, LEDs:LED_0603, B.Cu at (87.0, 58.5)
- added D1113: GRN, LEDs:LED_0603, B.Cu at (96.8, 58.7)
- added D1114: GRN, LEDs:LED_0603, B.Cu at (117.3, 58.5)
- added D1115: GRN, LEDs:LED_0603, B.Cu at (91.7, 58.5)
- added D1116: GRN, LEDs:LED_0603, B.Cu at (102.1, 58.5)
- added D1117: GRN, LEDs:LED_0603, B.Cu at (107.6, 58.5)
- added D1118: GRN, LEDs:LED_0603, B.Cu at (112.4, 58.5)
- added D1119: GRN, LEDs:LED_0603, B.Cu at (122.3, 58.5)
- added D1120: GRN, LEDs:LED_0603, B.Cu at (127.9, 58.5)
- added D1201: GRN, LEDs:LED_0603, B.Cu at (133.1, 58.5)
- added D1202: GRN, LEDs:LED_0603, B.Cu at (158.3, 58.5)
- added D1203: GRN, LEDs:LED_0603, B.Cu at (178.2, 58.5)
- added D1204: GRN, LEDs:LED_0603, B.Cu at (137.7, 58.5)
- added D1205: GRN, LEDs:LED_0603, B.Cu at (142.5, 58.5)
- added D1206: GRN, LEDs:LED_0603, B.Cu at (147.5, 58.5)
- added D1207: GRN, LEDs:LED_0603, B.Cu at (152.8, 58.7)
- added D1208: GRN, LEDs:LED_0603, B.Cu at (163.2, 58.5)
- added D1209: GRN, LEDs:LED_0603, B.Cu at (168.2, 58.5)
- added D1210: GRN, LEDs:LED_0603, B.Cu at (173.0, 58.5)
- added D1211: GRN, LEDs:LED_0603, B.Cu at (183.5, 58.5)
- added D1212: GRN, LEDs:LED_0603, B.Cu at (188.5, 58.5)
- added D1213: GRN, LEDs:LED_0603, B.Cu at (198.3, 58.7)
- added D1214: GRN, LEDs:LED_0603, B.Cu at (218.8, 58.5)
- added D1215: GRN, LEDs:LED_0603, B.Cu at (193.2, 58.5)
- added D1216: GRN, LEDs:LED_0603, B.Cu at (203.6, 58.5)
- added D1217: GRN, LEDs:LED_0603, B.Cu at (209.1, 58.5)
- added D1218: GRN, LEDs:LED_0603, B.Cu at (213.9, 58.5)
- added D1219: GRN, LEDs:LED_0603, B.Cu at (223.8, 58.5)
- added D1220: GRN, LEDs:LED_0603, B.Cu at (229.4, 58.5)
- added D1301: GRN, LEDs:LED_0603, B.Cu at (234.6, 58.5)
- added D1302: GRN, LEDs:LED_0603, B.Cu at (259.8, 58.5)
- added D1303: GRN, LEDs:LED_0603, B.Cu at (279.7, 58.5)
- added D1304: GRN, LEDs:LED_0603, B.Cu at (239.2, 58.5)
- added D1305: GRN, LEDs:LED_0603, B.Cu at (244.0, 58.5)
- added D1306: GRN, LEDs:LED_0603, B.Cu at (249.0, 58.5)
- added D1307: GRN, LEDs:LED_0603, B.Cu at (254.3, 58.7)
- added D1308: GRN, LEDs:LED_0603, B.Cu at (264.7, 58.5)
- added D1309: GRN, LEDs:LED_0603, B.Cu at (269.7, 58.5)
- added D1310: GRN, LEDs:LED_0603, B.Cu at (274.5, 58.5)
- added D1311: GRN, LEDs:LED_0603, B.Cu at (285.0, 58.5)
- added D1312: GRN, LEDs:LED_0603, B.Cu at (290.0, 58.5)
- added D1313: GRN, LEDs:LED_0603, B.Cu at (299.8, 58.7)
- added D1314: GRN, LEDs:LED_0603, B.Cu at (320.3, 58.5)
- added D1315: GRN, LEDs:LED_0603, B.Cu at (294.7, 58.5)
- added D1316: GRN, LEDs:LED_0603, B.Cu at (305.1, 58.5)
- added D1317: GRN, LEDs:LED_0603, B.Cu at (310.6, 58.5)
- added D1318: GRN, LEDs:LED_0603, B.Cu at (315.4, 58.5)
- added D1319: GRN, LEDs:LED_0603, B.Cu at (325.3, 58.5)
- added D1320: GRN, LEDs:LED_0603, B.Cu at (330.9, 58.5)
- added D1401: GRN, LEDs:LED_0603, B.Cu at (336.1, 58.5)
- added D1402: GRN, LEDs:LED_0603, B.Cu at (361.3, 58.5)
- added D1403: GRN, LEDs:LED_0603, B.Cu at (381.2, 58.5)
- added D1404: GRN, LEDs:LED_0603, B.Cu at (340.7, 58.5)
- added D1405: GRN, LEDs:LED_0603, B.Cu at (345.5, 58.5)
- added D1406: GRN, LEDs:LED_0603, B.Cu at (350.5, 58.5)
- added D1407: GRN, LEDs:LED_0603, B.Cu at (355.8, 58.7)
- added D1408: GRN, LEDs:LED_0603, B.Cu at (366.2, 58.5)
- added D1409: GRN, LEDs:LED_0603, B.Cu at (371.2, 58.5)
- added D1410: GRN, LEDs:LED_0603, B.Cu at (376.0, 58.5)
- added D1411: GRN, LEDs:LED_0603, B.Cu at (386.5, 58.5)
- added D1412: GRN, LEDs:LED_0603, B.Cu at (391.5, 58.5)
- added D1413: GRN, LEDs:LED_0603, B.Cu at (401.3, 58.7)
- added D1414: GRN, LEDs:LED_0603, B.Cu at (421.8, 58.5)
- added D1415: GRN, LEDs:LED_0603, B.Cu at (396.2, 58.5)
- added D1416: GRN, LEDs:LED_0603, B.Cu at (406.6, 58.5)
- added D1417: GRN, LEDs:LED_0603, B.Cu at (412.1, 58.5)
- added D1418: GRN, LEDs:LED_0603, B.Cu at (416.9, 58.5)
- added D1419: GRN, LEDs:LED_0603, B.Cu at (426.8, 58.5)
- added D1420: GRN, LEDs:LED_0603, B.Cu at (432.4, 58.5)
- added D1501: GRN, LEDs:LED_0603, B.Cu at (437.6, 58.5)
- added D1502: GRN, LEDs:LED_0603, B.Cu at (462.8, 58.5)
- added D1503: GRN, LEDs:LED_0603, B.Cu at (482.7, 58.5)
- added D1504: GRN, LEDs:LED_0603, B.Cu at (442.2, 58.5)
- added D1505: GRN, LEDs:LED_0603, B.Cu at (447.0, 58.5)
- added D1506: GRN, LEDs:LED_0603, B.Cu at (452.0, 58.5)
- added D1507: GRN, LEDs:LED_0603, B.Cu at (457.3, 58.7)
- added D1508: GRN, LEDs:LED_0603, B.Cu at (467.7, 58.5)
- added D1509: GRN, LEDs:LED_0603, B.Cu at (472.7, 58.5)
- added D1510: GRN, LEDs:LED_0603, B.Cu at (477.5, 58.5)
- added D1511: GRN, LEDs:LED_0603, B.Cu at (488.0, 58.5)
- added D1512: GRN, LEDs:LED_0603, B.Cu at (493.0, 58.5)
- added D1513: GRN, LEDs:LED_0603, B.Cu at (502.8, 58.7)
- added D1514: GRN, LEDs:LED_0603, B.Cu at (523.3, 58.5)
- added D1515: GRN, LEDs:LED_0603, B.Cu at (497.7, 58.5)
- added D1516: GRN, LEDs:LED_0603, B.Cu at (508.1, 58.5)
- added D1517: GRN, LEDs:LED_0603, B.Cu at (513.6, 58.5)
- added D1518: GRN, LEDs:LED_0603, B.Cu at (518.4, 58.5)
- added D1519: GRN, LEDs:LED_0603, B.Cu at (528.3, 58.5)
- added D1520: GRN, LEDs:LED_0603, B.Cu at (533.9, 58.5)
- added D1601: GRN, LEDs:LED_0603, B.Cu at (539.1, 58.5)
- added D1602: GRN, LEDs:LED_0603, B.Cu at (564.3, 58.5)
- added D1603: GRN, LEDs:LED_0603, B.Cu at (584.2, 58.5)
- added D1604: GRN, LEDs:LED_0603, B.Cu at (543.7, 58.5)
- added D1605: GRN, LEDs:LED_0603, B.Cu at (548.5, 58.5)
- added D1606: GRN, LEDs:LED_0603, B.Cu at (553.5, 58.5)
- added D1607: GRN, LEDs:LED_0603, B.Cu at (558.8, 58.7)
- added D1608: GRN, LEDs:LED_0603, B.Cu at (569.2, 58.5)
- added D1609: GRN, LEDs:LED_0603, B.Cu at (574.2, 58.5)
- added D1610: GRN, LEDs:LED_0603, B.Cu at (579.0, 58.5)
- added D1611: GRN, LEDs:LED_0603, B.Cu at (589.5, 58.5)
- added D1612: GRN, LEDs:LED_0603, B.Cu at (594.5, 58.5)
- added D1613: GRN, LEDs:LED_0603, B.Cu at (604.3, 58.7)
- added D1614: GRN, LEDs:LED_0603, B.Cu at (624.8, 58.5)
- added D1615: GRN, LEDs:LED_0603, B.Cu at (599.2, 58.5)
- added D1616: GRN, LEDs:LED_0603, B.Cu at (609.6, 58.5)
- added D1617: GRN, LEDs:LED_0603, B.Cu at (615.1, 58.5)
- added D1618: GRN, LEDs:LED_0603, B.Cu at (619.9, 58.5)
- added D1619: GRN, LEDs:LED_0603, B.Cu at (629.8, 58.5)
- added D1620: GRN, LEDs:LED_0603, B.Cu at (635.4, 58.5)
- added D1701: GRN, LEDs:LED_0603, B.Cu at (640.6, 58.5)
- added D1702: GRN, LEDs:LED_0603, B.Cu at (665.8, 58.5)
- added D1703: GRN, LEDs:LED_0603, B.Cu at (685.7, 58.5)
- added D1704: GRN, LEDs:LED_0603, B.Cu at (645.2, 58.5)
- added D1705: GRN, LEDs:LED_0603, B.Cu at (650.0, 58.5)
- added D1706: GRN, LEDs:LED_0603, B.Cu at (655.0, 58.5)
- added D1707: GRN, LEDs:LED_0603, B.Cu at (660.3, 58.7)
- added D1708: GRN, LEDs:LED_0603, B.Cu at (670.7, 58.5)
- added D1709: GRN, LEDs:LED_0603, B.Cu at (675.7, 58.5)
- added D1710: GRN, LEDs:LED_0603, B.Cu at (680.5, 58.5)
- added D1711: GRN, LEDs:LED_0603, B.Cu at (691.0, 58.5)
- added D1712: GRN, LEDs:LED_0603, B.Cu at (696.0, 58.5)
- added D1713: GRN, LEDs:LED_0603, B.Cu at (705.8, 58.7)
- added D1714: GRN, LEDs:LED_0603, B.Cu at (726.3, 58.5)
- added D1715: GRN, LEDs:LED_0603, B.Cu at (700.7, 58.5)
- added D1716: GRN, LEDs:LED_0603, B.Cu at (711.1, 58.5)
- added D1717: GRN, LEDs:LED_0603, B.Cu at (716.6, 58.5)
- added D1718: GRN, LEDs:LED_0603, B.Cu at (721.4, 58.5)
- added D1719: GRN, LEDs:LED_0603, B.Cu at (731.3, 58.5)
- added D1720: GRN, LEDs:LED_0603, B.Cu at (736.9, 58.5)
- added D1801: GRN, LEDs:LED_0603, B.Cu at (742.1, 58.5)
- added D1802: GRN, LEDs:LED_0603, B.Cu at (767.3, 58.5)
- added D1803: GRN, LEDs:LED_0603, B.Cu at (787.2, 58.5)
- added D1804: GRN, LEDs:LED_0603, B.Cu at (746.7, 58.5)
- added D1805: GRN, LEDs:LED_0603, B.Cu at (751.5, 58.5)
- added D1806: GRN, LEDs:LED_0603, B.Cu at (756.5, 58.5)
- added D1807: GRN, LEDs:LED_0603, B.Cu at (761.8, 58.7)
- added D1808: GRN, LEDs:LED_0603, B.Cu at (772.2, 58.5)
- added D1809: GRN, LEDs:LED_0603, B.Cu at (777.2, 58.5)
- added D1810: GRN, LEDs:LED_0603, B.Cu at (782.0, 58.5)
- added D1811: GRN, LEDs:LED_0603, B.Cu at (792.5, 58.5)
- added D1812: GRN, LEDs:LED_0603, B.Cu at (797.5, 58.5)
- added D1813: GRN, LEDs:LED_0603, B.Cu at (807.3, 58.7)
- added D1814: GRN, LEDs:LED_0603, B.Cu at (827.8, 58.5)
- added D1815: GRN, LEDs:LED_0603, B.Cu at (802.2, 58.5)
- added D1816: GRN, LEDs:LED_0603, B.Cu at (812.6, 58.5)
- added D1817: GRN, LEDs:LED_0603, B.Cu at (818.1, 58.5)
- added D1818: GRN, LEDs:LED_0603, B.Cu at (822.9, 58.5)
- added D1819: GRN, LEDs:LED_0603, B.Cu at (832.8, 58.5)
- added D1820: GRN, LEDs:LED_0603, B.Cu at (838.4, 58.5)
- added D1901: GRN, LEDs:LED_0603, B.Cu at (843.5, 58.7)
- added D1902: GRN, LEDs:LED_0603, B.Cu at (868.3, 58.8)
- added D1903: GRN, LEDs:LED_0603, B.Cu at (887.3, 58.8)
- added D1904: GRN, LEDs:LED_0603, B.Cu at (849.1, 58.8)
- added D1905: GRN, LEDs:LED_0603, B.Cu at (854.1, 58.8)
- added D1906: GRN, LEDs:LED_0603, B.Cu at (858.9, 58.8)
- added D1907: GRN, LEDs:LED_0603, B.Cu at (863.5, 58.8)
- added D1908: GRN, LEDs:LED_0603, B.Cu at (873.0, 58.8)
- added D1909: GRN, LEDs:LED_0603, B.Cu at (877.7, 58.8)
- added D1910: GRN, LEDs:LED_0603, B.Cu at (882.6, 58.8)
- added D1911: GRN, LEDs:LED_0603, B.Cu at (892.3, 58.8)
- added D1912: GRN, LEDs:LED_0603, B.Cu at (897.4, 58.8)
- added D1913: GRN, LEDs:LED_0603, B.Cu at (907.2, 58.8)
- added D1914: GRN, LEDs:LED_0603, B.Cu at (902.3, 58.8)
- added D1915: GRN, LEDs:LED_0603, B.Cu at (912.4, 58.9)
- added D1916: GRN, LEDs:LED_0603, B.Cu at (917.6, 58.8)
- added D301: GRN, LEDs:LED_0603, F.Cu at (133.1, 58.4)
- added D302: GRN, LEDs:LED_0603, F.Cu at (158.5, 58.5)
- added D303: GRN, LEDs:LED_0603, F.Cu at (178.5, 58.4)
- added D304: GRN, LEDs:LED_0603, F.Cu at (137.7, 58.4)
- added D305: GRN, LEDs:LED_0603, F.Cu at (142.8, 58.4)
- added D306: GRN, LEDs:LED_0603, F.Cu at (148.0, 58.4)
- added D307: GRN, LEDs:LED_0603, F.Cu at (153.1, 58.5)
- added D308: GRN, LEDs:LED_0603, F.Cu at (163.5, 58.5)
- added D309: GRN, LEDs:LED_0603, F.Cu at (168.3, 58.5)
- added D310: GRN, LEDs:LED_0603, F.Cu at (173.3, 58.4)
- added D311: GRN, LEDs:LED_0603, F.Cu at (183.8, 58.4)
- added D312: GRN, LEDs:LED_0603, F.Cu at (188.7, 58.5)
- added D313: GRN, LEDs:LED_0603, F.Cu at (198.5, 58.5)
- added D314: GRN, LEDs:LED_0603, F.Cu at (219.1, 58.5)
- added D315: GRN, LEDs:LED_0603, F.Cu at (193.4, 58.5)
- added D316: GRN, LEDs:LED_0603, F.Cu at (203.9, 58.5)
- added D317: GRN, LEDs:LED_0603, F.Cu at (209.3, 58.5)
- added D318: GRN, LEDs:LED_0603, F.Cu at (214.1, 58.5)
- added D319: GRN, LEDs:LED_0603, F.Cu at (224.1, 58.5)
- added D320: GRN, LEDs:LED_0603, F.Cu at (229.5, 58.5)
- added D401: GRN, LEDs:LED_0603, F.Cu at (234.6, 58.4)
- added D402: GRN, LEDs:LED_0603, F.Cu at (260.0, 58.5)
- added D403: GRN, LEDs:LED_0603, F.Cu at (280.0, 58.4)
- added D404: GRN, LEDs:LED_0603, F.Cu at (239.2, 58.4)
- added D405: GRN, LEDs:LED_0603, F.Cu at (244.3, 58.4)
- added D406: GRN, LEDs:LED_0603, F.Cu at (249.5, 58.4)
- added D407: GRN, LEDs:LED_0603, F.Cu at (254.6, 58.5)
- added D408: GRN, LEDs:LED_0603, F.Cu at (265.0, 58.5)
- added D409: GRN, LEDs:LED_0603, F.Cu at (269.8, 58.5)
- added D410: GRN, LEDs:LED_0603, F.Cu at (274.8, 58.4)
- added D411: GRN, LEDs:LED_0603, F.Cu at (285.3, 58.4)
- added D412: GRN, LEDs:LED_0603, F.Cu at (290.2, 58.5)
- added D413: GRN, LEDs:LED_0603, F.Cu at (300.0, 58.5)
- added D414: GRN, LEDs:LED_0603, F.Cu at (320.6, 58.5)
- added D415: GRN, LEDs:LED_0603, F.Cu at (294.9, 58.5)
- added D416: GRN, LEDs:LED_0603, F.Cu at (305.4, 58.5)
- added D417: GRN, LEDs:LED_0603, F.Cu at (310.8, 58.5)
- added D418: GRN, LEDs:LED_0603, F.Cu at (315.6, 58.5)
- added D419: GRN, LEDs:LED_0603, F.Cu at (325.6, 58.5)
- added D420: GRN, LEDs:LED_0603, F.Cu at (331.0, 58.5)
- added D501: GRN, LEDs:LED_0603, F.Cu at (336.1, 58.4)
- added D502: GRN, LEDs:LED_0603, F.Cu at (361.5, 58.5)
- added D503: GRN, LEDs:LED_0603, F.Cu at (381.5, 58.4)
- added D504: GRN, LEDs:LED_0603, F.Cu at (340.7, 58.4)
- added D505: GRN, LEDs:LED_0603, F.Cu at (345.8, 58.4)
- added D506: GRN, LEDs:LED_0603, F.Cu at (351.0, 58.4)
- added D507: GRN, LEDs:LED_0603, F.Cu at (356.1, 58.5)
- added D508: GRN, LEDs:LED_0603, F.Cu at (366.5, 58.5)
- added D509: GRN, LEDs:LED_0603, F.Cu at (371.3, 58.5)
- added D510: GRN, LEDs:LED_0603, F.Cu at (376.3, 58.4)
- added D511: GRN, LEDs:LED_0603, F.Cu at (386.8, 58.4)
- added D512: GRN, LEDs:LED_0603, F.Cu at (391.7, 58.5)
- added D513: GRN, LEDs:LED_0603, F.Cu at (401.5, 58.5)
- added D514: GRN, LEDs:LED_0603, F.Cu at (422.1, 58.5)
- added D515: GRN, LEDs:LED_0603, F.Cu at (396.4, 58.5)
- added D516: GRN, LEDs:LED_0603, F.Cu at (406.9, 58.5)
- added D517: GRN, LEDs:LED_0603, F.Cu at (412.3, 58.5)
- added D518: GRN, LEDs:LED_0603, F.Cu at (417.1, 58.5)
- added D519: GRN, LEDs:LED_0603, F.Cu at (427.1, 58.5)
- added D520: GRN, LEDs:LED_0603, F.Cu at (432.5, 58.5)
- added D601: GRN, LEDs:LED_0603, F.Cu at (437.6, 58.4)
- added D602: GRN, LEDs:LED_0603, F.Cu at (463.0, 58.5)
- added D603: GRN, LEDs:LED_0603, F.Cu at (483.0, 58.4)
- added D604: GRN, LEDs:LED_0603, F.Cu at (442.2, 58.4)
- added D605: GRN, LEDs:LED_0603, F.Cu at (447.3, 58.4)
- added D606: GRN, LEDs:LED_0603, F.Cu at (452.5, 58.4)
- added D607: GRN, LEDs:LED_0603, F.Cu at (457.6, 58.5)
- added D608: GRN, LEDs:LED_0603, F.Cu at (468.0, 58.5)
- added D609: GRN, LEDs:LED_0603, F.Cu at (472.8, 58.5)
- added D610: GRN, LEDs:LED_0603, F.Cu at (477.8, 58.4)
- added D611: GRN, LEDs:LED_0603, F.Cu at (488.3, 58.4)
- added D612: GRN, LEDs:LED_0603, F.Cu at (493.2, 58.5)
- added D613: GRN, LEDs:LED_0603, F.Cu at (503.0, 58.5)
- added D614: GRN, LEDs:LED_0603, F.Cu at (523.6, 58.5)
- added D615: GRN, LEDs:LED_0603, F.Cu at (497.9, 58.5)
- added D616: GRN, LEDs:LED_0603, F.Cu at (508.4, 58.5)
- added D617: GRN, LEDs:LED_0603, F.Cu at (513.8, 58.5)
- added D618: GRN, LEDs:LED_0603, F.Cu at (518.6, 58.5)
- added D619: GRN, LEDs:LED_0603, F.Cu at (528.6, 58.5)
- added D620: GRN, LEDs:LED_0603, F.Cu at (534.0, 58.5)
- added D701: GRN, LEDs:LED_0603, F.Cu at (539.1, 58.4)
- added D702: GRN, LEDs:LED_0603, F.Cu at (564.5, 58.5)
- added D703: GRN, LEDs:LED_0603, F.Cu at (584.5, 58.4)
- added D704: GRN, LEDs:LED_0603, F.Cu at (543.7, 58.4)
- added D705: GRN, LEDs:LED_0603, F.Cu at (548.8, 58.4)
- added D706: GRN, LEDs:LED_0603, F.Cu at (554.0, 58.4)
- added D707: GRN, LEDs:LED_0603, F.Cu at (559.1, 58.5)
- added D708: GRN, LEDs:LED_0603, F.Cu at (569.5, 58.5)
- added D709: GRN, LEDs:LED_0603, F.Cu at (574.3, 58.5)
- added D710: GRN, LEDs:LED_0603, F.Cu at (579.3, 58.4)
- added D711: GRN, LEDs:LED_0603, F.Cu at (589.8, 58.4)
- added D712: GRN, LEDs:LED_0603, F.Cu at (594.7, 58.5)
- added D713: GRN, LEDs:LED_0603, F.Cu at (604.5, 58.5)
- added D714: GRN, LEDs:LED_0603, F.Cu at (625.1, 58.5)
- added D715: GRN, LEDs:LED_0603, F.Cu at (599.4, 58.5)
- added D716: GRN, LEDs:LED_0603, F.Cu at (609.9, 58.5)
- added D717: GRN, LEDs:LED_0603, F.Cu at (615.3, 58.5)
- added D718: GRN, LEDs:LED_0603, F.Cu at (620.1, 58.5)
- added D719: GRN, LEDs:LED_0603, F.Cu at (630.1, 58.5)
- added D720: GRN, LEDs:LED_0603, F.Cu at (635.5, 58.5)
- added D801: GRN, LEDs:LED_0603, F.Cu at (640.6, 58.4)
- added D802: GRN, LEDs:LED_0603, F.Cu at (666.0, 58.5)
- added D803: GRN, LEDs:LED_0603, F.Cu at (686.0, 58.4)
- added D804: GRN, LEDs:LED_0603, F.Cu at (645.2, 58.4)
- added D805: GRN, LEDs:LED_0603, F.Cu at (650.3, 58.4)
- added D806: GRN, LEDs:LED_0603, F.Cu at (655.5, 58.4)
- added D807: GRN, LEDs:LED_0603, F.Cu at (660.6, 58.5)
- added D808: GRN, LEDs:LED_0603, F.Cu at (671.0, 58.5)
- added D809: GRN, LEDs:LED_0603, F.Cu at (675.8, 58.5)
- added D810: GRN, LEDs:LED_0603, F.Cu at (680.8, 58.4)
- added D811: GRN, LEDs:LED_0603, F.Cu at (691.3, 58.4)
- added D812: GRN, LEDs:LED_0603, F.Cu at (696.2, 58.5)
- added D813: GRN, LEDs:LED_0603, F.Cu at (706.0, 58.5)
- added D814: GRN, LEDs:LED_0603, F.Cu at (726.6, 58.5)
- added D815: GRN, LEDs:LED_0603, F.Cu at (700.9, 58.5)
- added D816: GRN, LEDs:LED_0603, F.Cu at (711.4, 58.5)
- added D817: GRN, LEDs:LED_0603, F.Cu at (716.8, 58.5)
- added D818: GRN, LEDs:LED_0603, F.Cu at (721.6, 58.5)
- added D819: GRN, LEDs:LED_0603, F.Cu at (731.6, 58.5)
- added D820: GRN, LEDs:LED_0603, F.Cu at (737.0, 58.5)
- added D901: GRN, LEDs:LED_0603, F.Cu at (742.1, 58.4)
- added D902: GRN, LEDs:LED_0603, F.Cu at (767.5, 58.5)
- added D903: GRN, LEDs:LED_0603, F.Cu at (787.5, 58.4)
- added D904: GRN, LEDs:LED_0603, F.Cu at (746.7, 58.4)
- added D905: GRN, LEDs:LED_0603, F.Cu at (751.8, 58.4)
- added D906: GRN, LEDs:LED_0603, F.Cu at (757.0, 58.4)
- added D907: GRN, LEDs:LED_0603, F.Cu at (762.1, 58.5)
- added D908: GRN, LEDs:LED_0603, F.Cu at (772.5, 58.5)
- added D909: GRN, LEDs:LED_0603, F.Cu at (777.3, 58.5)
- added D910: GRN, LEDs:LED_0603, F.Cu at (782.3, 58.4)
- added D911: GRN, LEDs:LED_0603, F.Cu at (792.8, 58.4)
- added D912: GRN, LEDs:LED_0603, F.Cu at (797.7, 58.5)
- added D913: GRN, LEDs:LED_0603, F.Cu at (807.5, 58.5)
- added D914: GRN, LEDs:LED_0603, F.Cu at (828.1, 58.5)
- added D915: GRN, LEDs:LED_0603, F.Cu at (802.4, 58.5)
- added D916: GRN, LEDs:LED_0603, F.Cu at (812.9, 58.5)
- added D917: GRN, LEDs:LED_0603, F.Cu at (818.3, 58.5)
- added D918: GRN, LEDs:LED_0603, F.Cu at (823.1, 58.5)
- added D919: GRN, LEDs:LED_0603, F.Cu at (833.1, 58.5)
- added D920: GRN, LEDs:LED_0603, F.Cu at (838.5, 58.5)
- added R1001: 442, Resistors_SMD:R_0603, F.Cu at (844.4, 56.0)
- added R1002: 442, Resistors_SMD:R_0603, F.Cu at (847.4, 56.0)
- added R1003: 442, Resistors_SMD:R_0603, F.Cu at (854.0, 56.0)
- added R1004: 442, Resistors_SMD:R_0603, F.Cu at (857.7, 56.0)
- added R1005: 442, Resistors_SMD:R_0603, F.Cu at (864.3, 56.0)
- added R1006: 442, Resistors_SMD:R_0603, F.Cu at (868.3, 56.0)
- added R1007: 442, Resistors_SMD:R_0603, F.Cu at (874.7, 56.0)
- added R1008: 442, Resistors_SMD:R_0603, F.Cu at (878.0, 56.0)
- added R1009: 442, Resistors_SMD:R_0603, F.Cu at (884.5, 56.0)
- added R1010: 442, Resistors_SMD:R_0603, F.Cu at (888.2, 56.0)
- added R1011: 442, Resistors_SMD:R_0603, F.Cu at (895.1, 56.0)
- added R1012: 442, Resistors_SMD:R_0603, F.Cu at (898.5, 56.0)
- added R1013: 0, Resistors_SMD:R_0603, F.Cu at (845.9, 58.4)
- added R1014: 0, Resistors_SMD:R_0603, F.Cu at (850.7, 58.5)
- added R1015: 0, Resistors_SMD:R_0603, F.Cu at (855.8, 58.4)
- added R1016: 0, Resistors_SMD:R_0603, F.Cu at (861.0, 58.5)
- added R1017: 0, Resistors_SMD:R_0603, F.Cu at (866.2, 58.5)
- added R1018: 0, Resistors_SMD:R_0603, F.Cu at (871.3, 58.5)
- added R1019: 0, Resistors_SMD:R_0603, F.Cu at (876.4, 58.5)
- added R1020: 0, Resistors_SMD:R_0603, F.Cu at (881.2, 58.4)
- added R1021: 0, Resistors_SMD:R_0603, F.Cu at (886.4, 58.4)
- added R1022: 0, Resistors_SMD:R_0603, F.Cu at (891.5, 58.4)
- added R1023: 0, Resistors_SMD:R_0603, F.Cu at (896.8, 58.5)
- added R1024: 0, Resistors_SMD:R_0603, F.Cu at (901.5, 58.5)
- added R1025: 0, Resistors_SMD:R_0603, F.Cu at (844.4, 60.8)
- added R1026: 0, Resistors_SMD:R_0603, F.Cu at (847.4, 60.8)
- added R1027: 0, Resistors_SMD:R_0603, F.Cu at (854.0, 60.8)
- added R1028: 0, Resistors_SMD:R_0603, F.Cu at (857.7, 60.8)
- added R1029: 0, Resistors_SMD:R_0603, F.Cu at (864.3, 60.8)
- added R1030: 0, Resistors_SMD:R_0603, F.Cu at (868.3, 60.8)
- added R1031: 0, Resistors_SMD:R_0603, F.Cu at (874.7, 60.8)
- added R1032: 0, Resistors_SMD:R_0603, F.Cu at (878.0, 60.8)
- added R1033: 0, Resistors_SMD:R_0603, F.Cu at (884.5, 60.8)
- added R1034: 0, Resistors_SMD:R_0603, F.Cu at (888.2, 60.8)
- added R1035: 0, Resistors_SMD:R_0603, F.Cu at (895.1, 60.8)
- added R1036: 0, Resistors_SMD:R_0603, F.Cu at (898.5, 60.8)
- added R1037: 442, Resistors_SMD:R_0603, F.Cu at (904.7, 56.0)
- added R1038: 442, Resistors_SMD:R_0603, F.Cu at (908.3, 56.0)
- added R1039: 442, Resistors_SMD:R_0603, F.Cu at (913.8, 56.0)
- added R1040: 442, Resistors_SMD:R_0603, F.Cu at (917.1, 56.0)
- added R1045: 0, Resistors_SMD:R_0603, F.Cu at (906.5, 58.5)
- added R1046: 0, Resistors_SMD:R_0603, F.Cu at (910.7, 58.7)
- added R1047: 0, Resistors_SMD:R_0603, F.Cu at (915.4, 58.5)
- added R1053: 0, Resistors_SMD:R_0603, F.Cu at (904.7, 60.8)
- added R1054: 0, Resistors_SMD:R_0603, F.Cu at (908.3, 60.8)
- added R1055: 0, Resistors_SMD:R_0603, F.Cu at (913.8, 60.8)
- added R1056: 0, Resistors_SMD:R_0603, F.Cu at (917.1, 60.8)
- added R1101: 442, Resistors_SMD:R_0603, B.Cu at (32.4, 56.3)
- added R1102: 442, Resistors_SMD:R_0603, B.Cu at (35.4, 56.3)
- added R1103: 442, Resistors_SMD:R_0603, B.Cu at (41.8, 56.1)
- added R1104: 442, Resistors_SMD:R_0603, B.Cu at (45.2, 56.1)
- added R1105: 442, Resistors_SMD:R_0603, B.Cu at (52.1, 56.1)
- added R1106: 442, Resistors_SMD:R_0603, B.Cu at (56.1, 56.1)
- added R1107: 442, Resistors_SMD:R_0603, B.Cu at (62.5, 56.1)
- added R1108: 442, Resistors_SMD:R_0603, B.Cu at (65.9, 56.1)
- added R1109: 442, Resistors_SMD:R_0603, B.Cu at (72.3, 56.1)
- added R1110: 442, Resistors_SMD:R_0603, B.Cu at (75.9, 56.1)
- added R1111: 442, Resistors_SMD:R_0603, B.Cu at (82.8, 56.1)
- added R1112: 442, Resistors_SMD:R_0603, B.Cu at (86.2, 56.1)
- added R1113: 0, Resistors_SMD:R_0603, B.Cu at (33.9, 58.5)
- added R1114: 0, Resistors_SMD:R_0603, B.Cu at (38.7, 58.5)
- added R1115: 0, Resistors_SMD:R_0603, B.Cu at (43.6, 58.5)
- added R1116: 0, Resistors_SMD:R_0603, B.Cu at (48.8, 58.5)
- added R1117: 0, Resistors_SMD:R_0603, B.Cu at (54.2, 58.7)
- added R1118: 0, Resistors_SMD:R_0603, B.Cu at (59.3, 58.5)
- added R1119: 0, Resistors_SMD:R_0603, B.Cu at (64.1, 58.5)
- added R1120: 0, Resistors_SMD:R_0603, B.Cu at (69.1, 58.5)
- added R1121: 0, Resistors_SMD:R_0603, B.Cu at (74.2, 58.7)
- added R1122: 0, Resistors_SMD:R_0603, B.Cu at (79.2, 58.5)
- added R1123: 0, Resistors_SMD:R_0603, B.Cu at (84.7, 58.5)
- added R1124: 0, Resistors_SMD:R_0603, B.Cu at (89.3, 58.5)
- added R1125: 0, Resistors_SMD:R_0603, B.Cu at (32.4, 61.0)
- added R1126: 0, Resistors_SMD:R_0603, B.Cu at (35.4, 61.0)
- added R1127: 0, Resistors_SMD:R_0603, B.Cu at (41.8, 61.0)
- added R1128: 0, Resistors_SMD:R_0603, B.Cu at (45.2, 61.0)
- added R1129: 0, Resistors_SMD:R_0603, B.Cu at (52.1, 61.1)
- added R1130: 0, Resistors_SMD:R_0603, B.Cu at (56.0, 61.1)
- added R1131: 0, Resistors_SMD:R_0603, B.Cu at (62.5, 61.2)
- added R1132: 0, Resistors_SMD:R_0603, B.Cu at (65.9, 61.2)
- added R1133: 0, Resistors_SMD:R_0603, B.Cu at (72.3, 61.2)
- added R1134: 0, Resistors_SMD:R_0603, B.Cu at (75.9, 61.2)
- added R1135: 0, Resistors_SMD:R_0603, B.Cu at (82.8, 61.2)
- added R1136: 0, Resistors_SMD:R_0603, B.Cu at (86.2, 61.2)
- added R1137: 442, Resistors_SMD:R_0603, B.Cu at (92.5, 56.1)
- added R1138: 442, Resistors_SMD:R_0603, B.Cu at (96.0, 56.1)
- added R1139: 442, Resistors_SMD:R_0603, B.Cu at (102.9, 56.1)
- added R1140: 442, Resistors_SMD:R_0603, B.Cu at (106.8, 56.1)
- added R1141: 442, Resistors_SMD:R_0603, B.Cu at (113.0, 56.1)
- added R1142: 442, Resistors_SMD:R_0603, B.Cu at (116.6, 56.1)
- added R1143: 442, Resistors_SMD:R_0603, B.Cu at (123.1, 56.1)
- added R1144: 442, Resistors_SMD:R_0603, B.Cu at (127.1, 56.1)
- added R1145: 0, Resistors_SMD:R_0603, B.Cu at (94.4, 58.5)
- added R1146: 0, Resistors_SMD:R_0603, B.Cu at (99.4, 58.7)
- added R1147: 0, Resistors_SMD:R_0603, B.Cu at (104.6, 58.5)
- added R1148: 0, Resistors_SMD:R_0603, B.Cu at (110.0, 58.5)
- added R1149: 0, Resistors_SMD:R_0603, B.Cu at (114.8, 58.5)
- added R1150: 0, Resistors_SMD:R_0603, B.Cu at (119.8, 58.5)
- added R1151: 0, Resistors_SMD:R_0603, B.Cu at (125.1, 58.5)
- added R1152: 0, Resistors_SMD:R_0603, B.Cu at (130.3, 58.5)
- added R1153: 0, Resistors_SMD:R_0603, B.Cu at (92.5, 61.2)
- added R1154: 0, Resistors_SMD:R_0603, B.Cu at (96.0, 61.2)
- added R1155: 0, Resistors_SMD:R_0603, B.Cu at (102.9, 61.2)
- added R1156: 0, Resistors_SMD:R_0603, B.Cu at (106.9, 61.2)
- added R1157: 0, Resistors_SMD:R_0603, B.Cu at (113.2, 61.2)
- added R1158: 0, Resistors_SMD:R_0603, B.Cu at (116.6, 61.2)
- added R1159: 0, Resistors_SMD:R_0603, B.Cu at (123.1, 61.2)
- added R1160: 0, Resistors_SMD:R_0603, B.Cu at (127.1, 61.2)
- added R1201: 442, Resistors_SMD:R_0603, B.Cu at (133.9, 56.3)
- added R1202: 442, Resistors_SMD:R_0603, B.Cu at (136.9, 56.3)
- added R1203: 442, Resistors_SMD:R_0603, B.Cu at (143.3, 56.1)
- added R1204: 442, Resistors_SMD:R_0603, B.Cu at (146.7, 56.1)
- added R1205: 442, Resistors_SMD:R_0603, B.Cu at (153.6, 56.1)
- added R1206: 442, Resistors_SMD:R_0603, B.Cu at (157.6, 56.1)
- added R1207: 442, Resistors_SMD:R_0603, B.Cu at (164.0, 56.1)
- added R1208: 442, Resistors_SMD:R_0603, B.Cu at (167.4, 56.1)
- added R1209: 442, Resistors_SMD:R_0603, B.Cu at (173.8, 56.1)
- added R1210: 442, Resistors_SMD:R_0603, B.Cu at (177.4, 56.1)
- added R1211: 442, Resistors_SMD:R_0603, B.Cu at (184.3, 56.1)
- added R1212: 442, Resistors_SMD:R_0603, B.Cu at (187.7, 56.1)
- added R1213: 0, Resistors_SMD:R_0603, B.Cu at (135.4, 58.5)
- added R1214: 0, Resistors_SMD:R_0603, B.Cu at (140.2, 58.5)
- added R1215: 0, Resistors_SMD:R_0603, B.Cu at (145.1, 58.5)
- added R1216: 0, Resistors_SMD:R_0603, B.Cu at (150.3, 58.5)
- added R1217: 0, Resistors_SMD:R_0603, B.Cu at (155.7, 58.7)
- added R1218: 0, Resistors_SMD:R_0603, B.Cu at (160.8, 58.5)
- added R1219: 0, Resistors_SMD:R_0603, B.Cu at (165.6, 58.5)
- added R1220: 0, Resistors_SMD:R_0603, B.Cu at (170.6, 58.5)
- added R1221: 0, Resistors_SMD:R_0603, B.Cu at (175.7, 58.7)
- added R1222: 0, Resistors_SMD:R_0603, B.Cu at (180.7, 58.5)
- added R1223: 0, Resistors_SMD:R_0603, B.Cu at (186.2, 58.5)
- added R1224: 0, Resistors_SMD:R_0603, B.Cu at (190.8, 58.5)
- added R1225: 0, Resistors_SMD:R_0603, B.Cu at (133.9, 61.0)
- added R1226: 0, Resistors_SMD:R_0603, B.Cu at (136.9, 61.0)
- added R1227: 0, Resistors_SMD:R_0603, B.Cu at (143.3, 61.0)
- added R1228: 0, Resistors_SMD:R_0603, B.Cu at (146.7, 61.0)
- added R1229: 0, Resistors_SMD:R_0603, B.Cu at (153.6, 61.1)
- added R1230: 0, Resistors_SMD:R_0603, B.Cu at (157.5, 61.1)
- added R1231: 0, Resistors_SMD:R_0603, B.Cu at (164.0, 61.2)
- added R1232: 0, Resistors_SMD:R_0603, B.Cu at (167.4, 61.2)
- added R1233: 0, Resistors_SMD:R_0603, B.Cu at (173.8, 61.2)
- added R1234: 0, Resistors_SMD:R_0603, B.Cu at (177.4, 61.2)
- added R1235: 0, Resistors_SMD:R_0603, B.Cu at (184.3, 61.2)
- added R1236: 0, Resistors_SMD:R_0603, B.Cu at (187.7, 61.2)
- added R1237: 442, Resistors_SMD:R_0603, B.Cu at (194.0, 56.1)
- added R1238: 442, Resistors_SMD:R_0603, B.Cu at (197.5, 56.1)
- added R1239: 442, Resistors_SMD:R_0603, B.Cu at (204.4, 56.1)
- added R1240: 442, Resistors_SMD:R_0603, B.Cu at (208.3, 56.1)
- added R1241: 442, Resistors_SMD:R_0603, B.Cu at (214.5, 56.1)
- added R1242: 442, Resistors_SMD:R_0603, B.Cu at (218.1, 56.1)
- added R1243: 442, Resistors_SMD:R_0603, B.Cu at (224.6, 56.1)
- added R1244: 442, Resistors_SMD:R_0603, B.Cu at (228.6, 56.1)
- added R1245: 0, Resistors_SMD:R_0603, B.Cu at (195.9, 58.5)
- added R1246: 0, Resistors_SMD:R_0603, B.Cu at (200.9, 58.7)
- added R1247: 0, Resistors_SMD:R_0603, B.Cu at (206.1, 58.5)
- added R1248: 0, Resistors_SMD:R_0603, B.Cu at (211.5, 58.5)
- added R1249: 0, Resistors_SMD:R_0603, B.Cu at (216.3, 58.5)
- added R1250: 0, Resistors_SMD:R_0603, B.Cu at (221.3, 58.5)
- added R1251: 0, Resistors_SMD:R_0603, B.Cu at (226.6, 58.5)
- added R1252: 0, Resistors_SMD:R_0603, B.Cu at (231.8, 58.5)
- added R1253: 0, Resistors_SMD:R_0603, B.Cu at (194.0, 61.2)
- added R1254: 0, Resistors_SMD:R_0603, B.Cu at (197.5, 61.2)
- added R1255: 0, Resistors_SMD:R_0603, B.Cu at (204.4, 61.2)
- added R1256: 0, Resistors_SMD:R_0603, B.Cu at (208.4, 61.2)
- added R1257: 0, Resistors_SMD:R_0603, B.Cu at (214.7, 61.2)
- added R1258: 0, Resistors_SMD:R_0603, B.Cu at (218.1, 61.2)
- added R1259: 0, Resistors_SMD:R_0603, B.Cu at (224.6, 61.2)
- added R1260: 0, Resistors_SMD:R_0603, B.Cu at (228.6, 61.2)
- added R1301: 442, Resistors_SMD:R_0603, B.Cu at (235.4, 56.3)
- added R1302: 442, Resistors_SMD:R_0603, B.Cu at (238.4, 56.3)
- added R1303: 442, Resistors_SMD:R_0603, B.Cu at (244.8, 56.1)
- added R1304: 442, Resistors_SMD:R_0603, B.Cu at (248.2, 56.1)
- added R1305: 442, Resistors_SMD:R_0603, B.Cu at (255.1, 56.1)
- added R1306: 442, Resistors_SMD:R_0603, B.Cu at (259.1, 56.1)
- added R1307: 442, Resistors_SMD:R_0603, B.Cu at (265.5, 56.1)
- added R1308: 442, Resistors_SMD:R_0603, B.Cu at (268.9, 56.1)
- added R1309: 442, Resistors_SMD:R_0603, B.Cu at (275.3, 56.1)
- added R1310: 442, Resistors_SMD:R_0603, B.Cu at (278.9, 56.1)
- added R1311: 442, Resistors_SMD:R_0603, B.Cu at (285.8, 56.1)
- added R1312: 442, Resistors_SMD:R_0603, B.Cu at (289.2, 56.1)
- added R1313: 0, Resistors_SMD:R_0603, B.Cu at (236.9, 58.5)
- added R1314: 0, Resistors_SMD:R_0603, B.Cu at (241.7, 58.5)
- added R1315: 0, Resistors_SMD:R_0603, B.Cu at (246.6, 58.5)
- added R1316: 0, Resistors_SMD:R_0603, B.Cu at (251.8, 58.5)
- added R1317: 0, Resistors_SMD:R_0603, B.Cu at (257.2, 58.7)
- added R1318: 0, Resistors_SMD:R_0603, B.Cu at (262.3, 58.5)
- added R1319: 0, Resistors_SMD:R_0603, B.Cu at (267.1, 58.5)
- added R1320: 0, Resistors_SMD:R_0603, B.Cu at (272.1, 58.5)
- added R1321: 0, Resistors_SMD:R_0603, B.Cu at (277.2, 58.7)
- added R1322: 0, Resistors_SMD:R_0603, B.Cu at (282.2, 58.5)
- added R1323: 0, Resistors_SMD:R_0603, B.Cu at (287.7, 58.5)
- added R1324: 0, Resistors_SMD:R_0603, B.Cu at (292.3, 58.5)
- added R1325: 0, Resistors_SMD:R_0603, B.Cu at (235.4, 61.0)
- added R1326: 0, Resistors_SMD:R_0603, B.Cu at (238.4, 61.0)
- added R1327: 0, Resistors_SMD:R_0603, B.Cu at (244.8, 61.0)
- added R1328: 0, Resistors_SMD:R_0603, B.Cu at (248.2, 61.0)
- added R1329: 0, Resistors_SMD:R_0603, B.Cu at (255.1, 61.1)
- added R1330: 0, Resistors_SMD:R_0603, B.Cu at (259.0, 61.1)
- added R1331: 0, Resistors_SMD:R_0603, B.Cu at (265.5, 61.2)
- added R1332: 0, Resistors_SMD:R_0603, B.Cu at (268.9, 61.2)
- added R1333: 0, Resistors_SMD:R_0603, B.Cu at (275.3, 61.2)
- added R1334: 0, Resistors_SMD:R_0603, B.Cu at (278.9, 61.2)
- added R1335: 0, Resistors_SMD:R_0603, B.Cu at (285.8, 61.2)
- added R1336: 0, Resistors_SMD:R_0603, B.Cu at (289.2, 61.2)
- added R1337: 442, Resistors_SMD:R_0603, B.Cu at (295.5, 56.1)
- added R1338: 442, Resistors_SMD:R_0603, B.Cu at (299.0, 56.1)
- added R1339: 442, Resistors_SMD:R_0603, B.Cu at (305.9, 56.1)
- added R1340: 442, Resistors_SMD:R_0603, B.Cu at (309.8, 56.1)
- added R1341: 442, Resistors_SMD:R_0603, B.Cu at (316.0, 56.1)
- added R1342: 442, Resistors_SMD:R_0603, B.Cu at (319.6, 56.1)
- added R1343: 442, Resistors_SMD:R_0603, B.Cu at (326.1, 56.1)
- added R1344: 442, Resistors_SMD:R_0603, B.Cu at (330.1, 56.1)
- added R1345: 0, Resistors_SMD:R_0603, B.Cu at (297.4, 58.5)
- added R1346: 0, Resistors_SMD:R_0603, B.Cu at (302.4, 58.7)
- added R1347: 0, Resistors_SMD:R_0603, B.Cu at (307.6, 58.5)
- added R1348: 0, Resistors_SMD:R_0603, B.Cu at (313.0, 58.5)
- added R1349: 0, Resistors_SMD:R_0603, B.Cu at (317.8, 58.5)
- added R1350: 0, Resistors_SMD:R_0603, B.Cu at (322.8, 58.5)
- added R1351: 0, Resistors_SMD:R_0603, B.Cu at (328.1, 58.5)
- added R1352: 0, Resistors_SMD:R_0603, B.Cu at (333.3, 58.5)
- added R1353: 0, Resistors_SMD:R_0603, B.Cu at (295.5, 61.2)
- added R1354: 0, Resistors_SMD:R_0603, B.Cu at (299.0, 61.2)
- added R1355: 0, Resistors_SMD:R_0603, B.Cu at (305.9, 61.2)
- added R1356: 0, Resistors_SMD:R_0603, B.Cu at (309.9, 61.2)
- added R1357: 0, Resistors_SMD:R_0603, B.Cu at (316.2, 61.2)
- added R1358: 0, Resistors_SMD:R_0603, B.Cu at (319.6, 61.2)
- added R1359: 0, Resistors_SMD:R_0603, B.Cu at (326.1, 61.2)
- added R1360: 0, Resistors_SMD:R_0603, B.Cu at (330.1, 61.2)
- added R1401: 442, Resistors_SMD:R_0603, B.Cu at (336.9, 56.3)
- added R1402: 442, Resistors_SMD:R_0603, B.Cu at (339.9, 56.3)
- added R1403: 442, Resistors_SMD:R_0603, B.Cu at (346.3, 56.1)
- added R1404: 442, Resistors_SMD:R_0603, B.Cu at (349.7, 56.1)
- added R1405: 442, Resistors_SMD:R_0603, B.Cu at (356.6, 56.1)
- added R1406: 442, Resistors_SMD:R_0603, B.Cu at (360.6, 56.1)
- added R1407: 442, Resistors_SMD:R_0603, B.Cu at (367.0, 56.1)
- added R1408: 442, Resistors_SMD:R_0603, B.Cu at (370.4, 56.1)
- added R1409: 442, Resistors_SMD:R_0603, B.Cu at (376.8, 56.1)
- added R1410: 442, Resistors_SMD:R_0603, B.Cu at (380.4, 56.1)
- added R1411: 442, Resistors_SMD:R_0603, B.Cu at (387.3, 56.1)
- added R1412: 442, Resistors_SMD:R_0603, B.Cu at (390.7, 56.1)
- added R1413: 0, Resistors_SMD:R_0603, B.Cu at (338.4, 58.5)
- added R1414: 0, Resistors_SMD:R_0603, B.Cu at (343.2, 58.5)
- added R1415: 0, Resistors_SMD:R_0603, B.Cu at (348.1, 58.5)
- added R1416: 0, Resistors_SMD:R_0603, B.Cu at (353.3, 58.5)
- added R1417: 0, Resistors_SMD:R_0603, B.Cu at (358.7, 58.7)
- added R1418: 0, Resistors_SMD:R_0603, B.Cu at (363.8, 58.5)
- added R1419: 0, Resistors_SMD:R_0603, B.Cu at (368.6, 58.5)
- added R1420: 0, Resistors_SMD:R_0603, B.Cu at (373.6, 58.5)
- added R1421: 0, Resistors_SMD:R_0603, B.Cu at (378.7, 58.7)
- added R1422: 0, Resistors_SMD:R_0603, B.Cu at (383.7, 58.5)
- added R1423: 0, Resistors_SMD:R_0603, B.Cu at (389.2, 58.5)
- added R1424: 0, Resistors_SMD:R_0603, B.Cu at (393.8, 58.5)
- added R1425: 0, Resistors_SMD:R_0603, B.Cu at (336.9, 61.0)
- added R1426: 0, Resistors_SMD:R_0603, B.Cu at (339.9, 61.0)
- added R1427: 0, Resistors_SMD:R_0603, B.Cu at (346.3, 61.0)
- added R1428: 0, Resistors_SMD:R_0603, B.Cu at (349.7, 61.0)
- added R1429: 0, Resistors_SMD:R_0603, B.Cu at (356.6, 61.1)
- added R1430: 0, Resistors_SMD:R_0603, B.Cu at (360.5, 61.1)
- added R1431: 0, Resistors_SMD:R_0603, B.Cu at (367.0, 61.2)
- added R1432: 0, Resistors_SMD:R_0603, B.Cu at (370.4, 61.2)
- added R1433: 0, Resistors_SMD:R_0603, B.Cu at (376.8, 61.2)
- added R1434: 0, Resistors_SMD:R_0603, B.Cu at (380.4, 61.2)
- added R1435: 0, Resistors_SMD:R_0603, B.Cu at (387.3, 61.2)
- added R1436: 0, Resistors_SMD:R_0603, B.Cu at (390.7, 61.2)
- added R1437: 442, Resistors_SMD:R_0603, B.Cu at (397.0, 56.1)
- added R1438: 442, Resistors_SMD:R_0603, B.Cu at (400.5, 56.1)
- added R1439: 442, Resistors_SMD:R_0603, B.Cu at (407.4, 56.1)
- added R1440: 442, Resistors_SMD:R_0603, B.Cu at (411.3, 56.1)
- added R1441: 442, Resistors_SMD:R_0603, B.Cu at (417.5, 56.1)
- added R1442: 442, Resistors_SMD:R_0603, B.Cu at (421.1, 56.1)
- added R1443: 442, Resistors_SMD:R_0603, B.Cu at (427.6, 56.1)
- added R1444: 442, Resistors_SMD:R_0603, B.Cu at (431.6, 56.1)
- added R1445: 0, Resistors_SMD:R_0603, B.Cu at (398.9, 58.5)
- added R1446: 0, Resistors_SMD:R_0603, B.Cu at (403.9, 58.7)
- added R1447: 0, Resistors_SMD:R_0603, B.Cu at (409.1, 58.5)
- added R1448: 0, Resistors_SMD:R_0603, B.Cu at (414.5, 58.5)
- added R1449: 0, Resistors_SMD:R_0603, B.Cu at (419.3, 58.5)
- added R1450: 0, Resistors_SMD:R_0603, B.Cu at (424.3, 58.5)
- added R1451: 0, Resistors_SMD:R_0603, B.Cu at (429.6, 58.5)
- added R1452: 0, Resistors_SMD:R_0603, B.Cu at (434.8, 58.5)
- added R1453: 0, Resistors_SMD:R_0603, B.Cu at (397.0, 61.2)
- added R1454: 0, Resistors_SMD:R_0603, B.Cu at (400.5, 61.2)
- added R1455: 0, Resistors_SMD:R_0603, B.Cu at (407.4, 61.2)
- added R1456: 0, Resistors_SMD:R_0603, B.Cu at (411.4, 61.2)
- added R1457: 0, Resistors_SMD:R_0603, B.Cu at (417.7, 61.2)
- added R1458: 0, Resistors_SMD:R_0603, B.Cu at (421.1, 61.2)
- added R1459: 0, Resistors_SMD:R_0603, B.Cu at (427.6, 61.2)
- added R1460: 0, Resistors_SMD:R_0603, B.Cu at (431.6, 61.2)
- added R1501: 442, Resistors_SMD:R_0603, B.Cu at (438.4, 56.3)
- added R1502: 442, Resistors_SMD:R_0603, B.Cu at (441.4, 56.3)
- added R1503: 442, Resistors_SMD:R_0603, B.Cu at (447.8, 56.1)
- added R1504: 442, Resistors_SMD:R_0603, B.Cu at (451.2, 56.1)
- added R1505: 442, Resistors_SMD:R_0603, B.Cu at (458.1, 56.1)
- added R1506: 442, Resistors_SMD:R_0603, B.Cu at (462.1, 56.1)
- added R1507: 442, Resistors_SMD:R_0603, B.Cu at (468.5, 56.1)
- added R1508: 442, Resistors_SMD:R_0603, B.Cu at (471.9, 56.1)
- added R1509: 442, Resistors_SMD:R_0603, B.Cu at (478.3, 56.1)
- added R1510: 442, Resistors_SMD:R_0603, B.Cu at (481.9, 56.1)
- added R1511: 442, Resistors_SMD:R_0603, B.Cu at (488.8, 56.1)
- added R1512: 442, Resistors_SMD:R_0603, B.Cu at (492.2, 56.1)
- added R1513: 0, Resistors_SMD:R_0603, B.Cu at (439.9, 58.5)
- added R1514: 0, Resistors_SMD:R_0603, B.Cu at (444.7, 58.5)
- added R1515: 0, Resistors_SMD:R_0603, B.Cu at (449.6, 58.5)
- added R1516: 0, Resistors_SMD:R_0603, B.Cu at (454.8, 58.5)
- added R1517: 0, Resistors_SMD:R_0603, B.Cu at (460.2, 58.7)
- added R1518: 0, Resistors_SMD:R_0603, B.Cu at (465.3, 58.5)
- added R1519: 0, Resistors_SMD:R_0603, B.Cu at (470.1, 58.5)
- added R1520: 0, Resistors_SMD:R_0603, B.Cu at (475.1, 58.5)
- added R1521: 0, Resistors_SMD:R_0603, B.Cu at (480.2, 58.7)
- added R1522: 0, Resistors_SMD:R_0603, B.Cu at (485.2, 58.5)
- added R1523: 0, Resistors_SMD:R_0603, B.Cu at (490.7, 58.5)
- added R1524: 0, Resistors_SMD:R_0603, B.Cu at (495.3, 58.5)
- added R1525: 0, Resistors_SMD:R_0603, B.Cu at (438.4, 61.0)
- added R1526: 0, Resistors_SMD:R_0603, B.Cu at (441.4, 61.0)
- added R1527: 0, Resistors_SMD:R_0603, B.Cu at (447.8, 61.0)
- added R1528: 0, Resistors_SMD:R_0603, B.Cu at (451.2, 61.0)
- added R1529: 0, Resistors_SMD:R_0603, B.Cu at (458.1, 61.1)
- added R1530: 0, Resistors_SMD:R_0603, B.Cu at (462.0, 61.1)
- added R1531: 0, Resistors_SMD:R_0603, B.Cu at (468.5, 61.2)
- added R1532: 0, Resistors_SMD:R_0603, B.Cu at (471.9, 61.2)
- added R1533: 0, Resistors_SMD:R_0603, B.Cu at (478.3, 61.2)
- added R1534: 0, Resistors_SMD:R_0603, B.Cu at (481.9, 61.2)
- added R1535: 0, Resistors_SMD:R_0603, B.Cu at (488.8, 61.2)
- added R1536: 0, Resistors_SMD:R_0603, B.Cu at (492.2, 61.2)
- added R1537: 442, Resistors_SMD:R_0603, B.Cu at (498.5, 56.1)
- added R1538: 442, Resistors_SMD:R_0603, B.Cu at (502.0, 56.1)
- added R1539: 442, Resistors_SMD:R_0603, B.Cu at (508.9, 56.1)
- added R1540: 442, Resistors_SMD:R_0603, B.Cu at (512.8, 56.1)
- added R1541: 442, Resistors_SMD:R_0603, B.Cu at (519.0, 56.1)
- added R1542: 442, Resistors_SMD:R_0603, B.Cu at (522.6, 56.1)
- added R1543: 442, Resistors_SMD:R_0603, B.Cu at (529.1, 56.1)
- added R1544: 442, Resistors_SMD:R_0603, B.Cu at (533.1, 56.1)
- added R1545: 0, Resistors_SMD:R_0603, B.Cu at (500.4, 58.5)
- added R1546: 0, Resistors_SMD:R_0603, B.Cu at (505.4, 58.7)
- added R1547: 0, Resistors_SMD:R_0603, B.Cu at (510.6, 58.5)
- added R1548: 0, Resistors_SMD:R_0603, B.Cu at (516.0, 58.5)
- added R1549: 0, Resistors_SMD:R_0603, B.Cu at (520.8, 58.5)
- added R1550: 0, Resistors_SMD:R_0603, B.Cu at (525.8, 58.5)
- added R1551: 0, Resistors_SMD:R_0603, B.Cu at (531.1, 58.5)
- added R1552: 0, Resistors_SMD:R_0603, B.Cu at (536.3, 58.5)
- added R1553: 0, Resistors_SMD:R_0603, B.Cu at (498.5, 61.2)
- added R1554: 0, Resistors_SMD:R_0603, B.Cu at (502.0, 61.2)
- added R1555: 0, Resistors_SMD:R_0603, B.Cu at (508.9, 61.2)
- added R1556: 0, Resistors_SMD:R_0603, B.Cu at (512.9, 61.2)
- added R1557: 0, Resistors_SMD:R_0603, B.Cu at (519.2, 61.2)
- added R1558: 0, Resistors_SMD:R_0603, B.Cu at (522.6, 61.2)
- added R1559: 0, Resistors_SMD:R_0603, B.Cu at (529.1, 61.2)
- added R1560: 0, Resistors_SMD:R_0603, B.Cu at (533.1, 61.2)
- added R1601: 442, Resistors_SMD:R_0603, B.Cu at (539.9, 56.3)
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Connections:
- R252 pad 1: /Front1/BLOCK_OUT -> /Front2/BLOCK_IN
Routing:
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- added copper zone on B.Cu, net GND
- added copper zone on F.Cu, net GND
- added copper zone on B.Cu, net VDD
- added copper zone on F.Cu, net VDD
Other:
- outline, holes or cut-outs redrawn
- board text added: "+"
- board text added: "-"
- board text added: ".062 in. nominal"
- board text added: "1 oz copper"
- board text added: "FR4"
