File: SBR001-202.sch (KiCad schematic (older format))
At the start: 0 parts

Commit message: Schematic and layout complete and ready for review
Connections:
- wire segments 4 -> 22
- no-connect marks 1 -> 0
Other:
- note added: "BACK SIDE"
- note added: "FRONT SIDE"
