File: block-of-20-LEDs.sch (KiCad schematic (older format))
At the start: 80 parts

Commit message: Schematic and layout complete and ready for review
Parts:
- removed R222: 0, Resistors_SMD:R_0603, symbol R
- added R322: 0, Resistors_SMD:R_0603, symbol R
- renumbered D201 to D301, D202 to D302, D203 to D303, D204 to D304, D205 to D305, D206 to D306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
Connections:
- net at D311.2 (A), R311.2: now also R322.1
- net at D303.1 (K), R334.1: now also R322.2
